File: Schematic/sigma_delta_v1_0.brd (EAGLE design)
At the start: 120 x 70 mm, 64 parts, among them IC1 LM50, IC2 MC78M12CDTG, IC3 UA78M33DCY, IC4 LM50, IC5 ACPL-064L-000E, J1 SJ1-3523N, Q3 IRF3707S, Q4 IRF3707S, Q5 BSD223P, X1 1751251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

Commit message: adapted wireing width of power stage and exchanged bootstrap capacitor
Parts:
- C1: device rcl:C2220K -> rcl:C0805K
- C5: value (none) -> 330nF
- F1, F2, F3: value (none) -> 5A
- SJ2: device jumper:SJ_2 -> jumper:SJ_2W
- moved C1 4.77 mm to (40.1, 15.2)
- moved D1 3.76 mm to (37.6, 18.5), turned to 90 degrees
- moved F1 0.25 mm to (15.2, 52.3)
Routing:
- net VCC_MID: track 138.4 -> 119.5 mm
- net N$17: track 18.0 -> 10.8 mm
- net AGND_FPGA: track 149.8 -> 154.6 mm
- net N$10: track 41.2 -> 36.4 mm, vias 2 -> 0
- net AVCC_FPGA: track 128.2 -> 132.8 mm
- net H_BRIDGE_MID: track 105.7 -> 101.2 mm
- net VCC_HI: track 77.3 -> 78.6 mm
- net N$24: track 8.09 -> 7.29 mm
- net N$32: track 91.5 -> 92.3 mm
- net N$23: track 106.1 -> 106.9 mm
- net VCC_12: track 55.7 -> 55.1 mm
- net GND: vias 57 -> 76
- added copper zone on layer 1, net VCC_MID

Commit message: ERC and DRC done. Ready for production.
Parts:
- C1: value (none) -> 4.7µ
- C4: value (none) -> 100n
- moved C8 2.24 mm to (36.8, 27.4), turned to 0 degrees
- moved C4 0.76 mm to (48.5, 16.2)
Routing:
- net N$29: track 18.6 -> 21.1 mm
- net VCC_3.3: track 60.1 -> 59.2 mm
- net VCC_12: track 55.1 -> 54.3 mm
- net GND: vias 76 -> 82
