File: Schematic/sigma_delta_v1_0.brd (EAGLE design)
At the start: 120 x 70 mm, 64 parts, among them IC1 LM50, IC2 MC78M12CDTG, IC3 UA78M33DCY, IC4 LM50, IC5 ACPL-064L-000E, J1 SJ1-3523N, Q3 IRF3707S, Q4 IRF3707S, Q5 BSD223P, X1 1751251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

Commit message: generated gerber files for manufacturing
Routing:
- net GND: vias 82 -> 80
Other:
- board text added: "El Amplificator"

Commit message: reworked gerber files
Parts:
- moved J1 0.11 mm to (116.5, 35.1)
Changed lines of the file:
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@@
 <hole x="7" y="63" drill="3.2"/>
 <hole x="7" y="7" drill="3.2"/>
-<text x="18.0574" y="55.864115625" size="1.27" layer="25" distance="90">El Amplificator</text>
+<text x="16.0254" y="55.610115625" size="1.27" layer="25" distance="90">El Amplificator</text>
 <rectangle x1="19.6977" y1="57.797696875" x2="27.3177" y2="57.812934375" layer="25"/>
 <rectangle x1="19.667221875" y1="57.812934375" x2="27.348178125" y2="57.828171875" layer="25"/>
@@
 <attribute name="VALUE" x="16.51" y="47.446" size="1.27" layer="27" rot="R180"/>
 </element>
-<element name="J1" library="SamacSys_Parts" package="SJ13523N" value="SJ1-3523N" x="116.586" y="35" smashed="yes" rot="R180">
-<attribute name="DESCRIPTION" value="Phone Connectors 3.5 MM AUDIO JACK" x="116.586" y="35" size="1.778" layer="27" rot="R180" display="off"/>
-<attribute name="HEIGHT" value="5.5mm" x="116.586" y="35" size="1.778" layer="27" rot="R180" display="off"/>
-<attribute name="MOUSER_PART_NUMBER" value="490-SJ1-3523N" x="116.586" y="35" size="1.778" layer="27" rot="R180" display="off"/>
-<attribute name="MOUSER_PRICE-STOCK" value="https://www.mouser.co.uk/ProductDetail/CUI-Devices/SJ1-3523N?qs=WyjlAZoYn50aNl0vAhb3Tg%3D%3D" x="116.586" y="35" size="1.778" layer="27" rot="R180" display="off"/>
-<attribute name="MANUFACTURER_NAME" value="CUI Devices" x="116.586" y="35" size="1.778" layer="27" rot="R180" display="off"/>
-<attribute name="MANUFACTURER_PART_NUMBER" value="SJ1-3523N" x="116.586" y="35" size="1.778" layer="27" rot="R180" display="off"/>
-<attribute name="NAME" x="111.449" y="27.38" size="1.27" layer="25" rot="R180" align="center"/>
-<attribute name="VALUE" x="112.211" y="35" size="1.27" layer="27" rot="R180" align="center"/>
+<element name="J1" library="SamacSys_Parts" package="SJ13523N" value="SJ1-3523N" x="116.4844" y="35.0508" smashed="yes" rot="R180">
+<attribute name="DESCRIPTION" value="Phone Connectors 3.5 MM AUDIO JACK" x="116.4844" y="35.0508" size="1.778" layer="27" rot="R180" display="off"/>
+<attribute name="HEIGHT" value="5.5mm" x="116.4844" y="35.0508" size="1.778" layer="27" rot="R180" display="off"/>
+<attribute name="MOUSER_PART_NUMBER" value="490-SJ1-3523N" x="116.4844" y="35.0508" size="1.778" layer="27" rot="R180" display="off"/>
+<attribute name="MOUSER_PRICE-STOCK" value="https://www.mouser.co.uk/ProductDetail/CUI-Devices/SJ1-3523N?qs=WyjlAZoYn50aNl0vAhb3Tg%3D%3D" x="116.4844" y="35.0508" size="1.778" layer="27" rot="R180" display="off"/>
+<attribute name="MANUFACTURER_NAME" value="CUI Devices" x="116.4844" y="35.0508" size="1.778" layer="27" rot="R180" display="off"/>
+<attribute name="MANUFACTURER_PART_NUMBER" value="SJ1-3523N" x="116.4844" y="35.0508" size="1.778" layer="27" rot="R180" display="off"/>
+<attribute name="NAME" x="111.3474" y="27.4308" size="1.27" layer="25" rot="R180" align="center"/>
+<attribute name="VALUE" x="112.1094" y="35.0508" size="1.27" layer="27" rot="R180" align="center"/>
 </element>
 <element name="U$4" library="SamacSys_Parts" package="SOT65P210X100-6N" value="BSD235N" x="26.416" y="30.936" smashed="yes" rot="MR270">
@@
 <contactref element="J1" pad="3"/>
 <contactref element="SJ2" pad="3"/>
-<wire x1="107.086" y1="30" x2="102.9944" y2="30" width="1.778" layer="16"/>
+<wire x1="106.9844" y1="30.0508" x2="102.9944" y2="30" width="1.778" layer="16"/>
 <wire x1="102.9944" y1="30" x2="101.346" y2="31.6484" width="1.778" layer="16"/>
 <wire x1="101.346" y1="31.6484" x2="101.346" y2="31.9786" width="1.778" layer="16"/>
@@
 <contactref element="J1" pad="2"/>
 <contactref element="SJ2" pad="1"/>
-<wire x1="107.086" y1="40" x2="102.6618" y2="40" width="1.778" layer="16"/>
+<wire x1="106.9844" y1="40.0508" x2="102.6618" y2="40" width="1.778" layer="16"/>
 <wire x1="102.6618" y1="40" x2="101.346" y2="38.6842" width="1.778" layer="16"/>
 <wire x1="101.346" y1="38.6842" x2="101.346" y2="38.1762" width="1.778" layer="16"/>
